File: atmel_sol/bal_part.brd (EAGLE design)
At the start: 42.2 x 34.9 mm, 61 parts, among them Q1 BSS123, Q2 BSS123, Q3 BSS123, Q4 BSS123, Q5 BSS123, Q6 BSS123

Commit message: second edit
Parts:
- removed C7: (no value), rcl:C0805K
- removed JP1, JP2, JP3, JP4, JP5, JP6, JP7: (no value), pinhead:1X01
- removed R36: (no value), rcl:0411V
- added F1: NTCTHERMISTOR1206, SparkFun-PowerIC:PTC-1206
- added SJ1: JUMPER-PAD-3-NOFULL_BOX_SILK, SparkFun-Passives:PAD-JUMPER-3-NO_YES_SILK_FULL_BOX
- C1, C2, C3, C4, C5, C6: device rcl:C0805K -> resistor:C0805
- R10, R15, R20, R30, R31, R32, R33, R34, R35, R5: device rcl:R1206 -> resistor:R0805
- R25: device rcl:0411V -> resistor:R0805
- R26, R27, R28, R29: device rcl:0411V -> rcl:R1206
- moved Q1 35.1 mm to (38.0, 26.1), flipped to the bottom, turned to 0 degrees
- moved Q6 34.6 mm to (4.40, 26.0), flipped to the bottom, turned to 0 degrees
- moved R1 33.4 mm to (38.3, 23.0)
- moved R2 33.4 mm to (38.3, 25.6)
- moved R3 33.4 mm to (38.3, 28.1)
- moved R4 33.4 mm to (38.3, 30.7)
- moved R29 31.0 mm to (4.60, 23.0), turned to 0 degrees
- moved R35 28.7 mm to (8.80, 7.60), turned to 180 degrees
- moved U$1 28.6 mm to (19.6, 10.8), turned to 270 degrees
- moved R22 27.0 mm to (11.4, 30.6)
- moved R5 26.9 mm to (38.0, 23.0), flipped to the bottom, turned to 180 degrees
- moved R21 26.2 mm to (11.4, 25.4)
- moved R23 25.8 mm to (11.4, 28.2)
- moved R24 25.7 mm to (11.4, 23.0)
- moved R28 25.6 mm to (4.60, 25.6), turned to 0 degrees
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Connections:
- removed net D5: C4.1, C5.2, R31.2
- removed net N$20: Q3.1, R32.1
- removed net N$21: Q4.1, R33.1
- removed net N$22: Q5.1, R34.1
- removed net N$23: Q6.1, R35.1
- removed net N$24: C5.1, C6.2, R30.2
- removed net N$26: C3.1, C4.2, R32.2
- removed net N$27: C2.1, C3.2, R33.2
- removed net N$28: C1.1, C2.2, R34.2
- removed net N$29: C1.2, C7.2, R35.2
- new net CELL0: C6.2, Q6.2, R31.1
- new net CLK: U$1.P12
- new net CLK_OUT: U$1.P43
- new net CS_N: U$1.P13
- new net CS_N_OUT: U$1.P42
- new net DISCH1: R30.1, U$1.P9
- new net DISCH2: R25.1, U$1.P7
- new net DISCH3: R20.1, U$1.P5
- new net DISCH4: R15.1, U$1.P3
- new net DISCH5: R10.1, U$1.P1
- new net DISCH6: R5.1, U$1.P47
- new net IRQ: U$1.P11
- new net IRQ_IN: U$1.P44
- new net MISO: U$1.P16
- new net MISO_IN: U$1.P39
- new net MOSI: U$1.P15
- new net MOSI_OUT: U$1.P40
- new net N$10: Q5.1, R25.2
- new net N$12: Q6.1, R30.2
- new net N$3: Q2.3, R6.1, R7.1, R8.1, R9.1
- new net N$5: Q3.3, R11.1, R12.1, R13.1, R14.1
- new net N$7: Q4.3, R16.1, R17.1, R18.1, R19.1
- new net SCK: U$1.P14
- new net SCK_OUT: U$1.P41
- new net VDD: SJ1.3
- net CELL1: now also C5.2, C6.1, Q5.2, R26.2, R27.2, R28.2, R29.2, U$1.P8; no longer JP6.1, R21.2, R22.2, R23.2, R24.2, R29.1
- net CELL2: now also C4.2, C5.1, Q4.2, R21.2, R22.2, R23.2, R24.2, U$1.P6; no longer JP5.1, R17.2, R18.2, R19.2, R20.2, R28.1
- net CELL3: now also C3.2, C4.1, Q3.2, R17.2, R18.2, R19.2, U$1.P4; no longer JP4.1, R13.2, R14.2, R15.2, R27.1
- net CELL4: now also C2.2, C3.1, Q2.2, R13.2, R14.2, U$1.P2; no longer JP3.1, R10.2, R26.1, R9.2
- net CELL5: now also C1.2, C2.1, Q1.2, R9.2, U$1.P48; no longer JP2.1, R25.1, R5.2
- net CELL6: now also C1.1, R32.2, U$1.P46; no longer JP1.1, R36.1
- net GND: now also F1.2, R35.2, SJ1.1, U$1.P19, U$1.P20, U$1.P21, U$1.P22, U$1.P24, U$1.P27, U$1.P28; no longer C7.1, JP7.1, Q6.2
- net N$11: now also R26.1, R27.1, R28.1, R29.1; no longer R21.1, R22.1, R23.1, R24.1
- net N$13: now also R31.2, U$1.P10; no longer Q2.2, R26.2
- net N$14: now also R32.1, U$1.P45; no longer Q3.2, R27.2
- net N$15: now also R33.2, R34.2, U$1.P31; no longer Q4.2, R28.2
- net N$16: now also R33.1, U$1.P30; no longer Q5.2, R29.2
- net N$17: now also F1.1, R34.1, U$1.P29; no longer Q1.1, R30.1
- net N$18: now also R35.1, U$1.P32; no longer Q1.2, R25.2
- net N$19: now also SJ1.2, U$1.P17; no longer Q2.1, R31.1
- net N$2: now also Q1.1, R5.2; no longer C6.1, R36.2
- net N$4: now also Q2.1, R10.2; no longer Q2.3, R5.1, R6.1, R7.1, R8.1
- net N$6: now also Q3.1, R15.2; no longer Q3.3, R10.1, R11.1, R12.1, R9.1
- net N$8: now also Q4.1, R20.2; no longer Q4.3, R13.1, R14.1, R15.1, R16.1
- net N$9: now also R21.1, R22.1, R23.1, R24.1; no longer R17.1, R18.1, R19.1, R20.1
Routing:
- net DISCH1: track 0.00 -> 22.8 mm, vias 0 -> 1
- net GND: track 41.5 -> 21.0 mm
- net DISCH6: track 0.00 -> 19.9 mm, vias 0 -> 1
- net N$14: track 2.73 -> 22.5 mm
- net N$13: track 2.73 -> 21.2 mm
- net DISCH2: track 0.00 -> 17.3 mm, vias 0 -> 1
- net CELL6: track 16.3 -> 31.8 mm
- net MISO_IN: track 0.00 -> 14.7 mm
- net CLK_OUT: track 0.00 -> 14.7 mm
- net SCK_OUT: track 0.00 -> 14.7 mm
- net MOSI_OUT: track 0.00 -> 14.6 mm
- net IRQ_IN: track 0.00 -> 14.6 mm
- net CS_N_OUT: track 0.00 -> 14.6 mm
- net N$5: track 0.00 -> 14.4 mm, vias 0 -> 1
- net N$3: track 0.00 -> 14.3 mm, vias 0 -> 1
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Other:
- board size 42.2 x 34.9 mm -> 42.2 x 39.3 mm

Commit message: first working prototype
Parts:
- added R36: (no value), resistor:R0805
- added U$2: TCMT1103-OPTO, SparkFun-DiscreteSemi:SSOP-4
- added X1, X2: FH12-12S-0.5SH, con-hirose:FH12-12S-0.5SH
- moved R34 8.04 mm to (12.8, 2.40), turned to 270 degrees
- moved R33 6.62 mm to (14.8, 2.40), turned to 270 degrees
- moved R35 2.33 mm to (10.8, 6.40), turned to 90 degrees
- moved H3 0.40 mm to (38.3, 3.17)
- moved H4 0.40 mm to (38.3, 36.1)
Connections:
- removed net N$14: R32.1, U$1.P45
- new net OPTO_HI: U$2.1, X1.11, X2.11
- new net OPTO_LOW: U$2.2, X1.12, X2.12
- new net PD_N: U$1.P38, U$2.3
- new net VDDHV: R32.1, U$1.P45, U$2.4
- new net VDDHVM: U$1.P36, X2.7
- new net VDDHVP: U$1.P37, X1.7
- net CELL0: now also R36.2
- net CLK: now also X2.2
- net CLK_OUT: now also X1.2
- net CS_N: now also X2.3
- net CS_N_OUT: now also X1.3
- net GND: now also R36.1
- net IRQ: now also X2.1
- net IRQ_IN: now also X1.1
- net MISO: now also X2.6
- net MISO_IN: now also X1.6
- net MOSI: now also X2.5
- net MOSI_OUT: now also X1.5
- net SCK: now also X2.4
- net SCK_OUT: now also X1.4
- net VDD: now also U$1.P23, U$1.P26, U$1.P34
Routing:
- net OPTO_LOW: track 0.00 -> 47.9 mm, vias 0 -> 2
- net OPTO_HI: track 0.00 -> 45.9 mm, vias 0 -> 2
- net N$17: track 13.2 -> 54.9 mm, vias 0 -> 1
- net GND: track 21.0 -> 61.7 mm, vias 0 -> 1
- net VDDHV: track 0.00 -> 24.3 mm
- net N$14: track 22.5 -> 0.00 mm
- net VDDHVM: track 0.00 -> 21.8 mm, vias 0 -> 2
- net N$18: track 0.00 -> 18.1 mm, vias 0 -> 2
- net VDD: track 0.00 -> 17.6 mm, vias 0 -> 2
- net PD_N: track 0.00 -> 16.1 mm
- net VDDHVP: track 0.00 -> 15.5 mm, vias 0 -> 1
- net N$15: track 0.00 -> 12.4 mm
- net N$16: track 0.00 -> 7.19 mm
- net CELL0: track 11.4 -> 16.6 mm
- net MOSI: track 6.87 -> 10.0 mm
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Other:
- board size 42.2 x 39.3 mm -> 41.4 x 39.3 mm
