File: atmel_sol/bal_part.sch (EAGLE design)
At the start: 61 parts, among them Q1 BSS123, Q2 BSS123, Q3 BSS123, Q4 BSS123, Q5 BSS123, Q6 BSS123

Commit message: second edit
Parts:
- removed C7: (no value), rcl:C-EUC0805K
- removed JP1, JP2, JP3, JP4, JP5, JP6, JP7: (no value), pinhead:PINHD-1X1
- removed R36: (no value), rcl:R-EU_0411/3V
- added F1: NTCTHERMISTOR1206, SparkFun-PowerIC:PTCTHERMISTOR1206
- added SJ1: JUMPER-PAD-3-NOFULL_BOX_SILK, SparkFun-Passives:JUMPER-PAD-3-NOFULL_BOX_SILK
- C1, C2, C3, C4, C5, C6: device rcl:C-EUC0805K -> resistor:C-EUC0805
- R10, R15, R20, R30, R31, R32, R33, R34, R35, R5: device rcl:R-EU_R1206 -> resistor:R-EU_R0805
- R25: device rcl:R-EU_0411/3V -> resistor:R-EU_R0805
- R26, R27, R28, R29: device rcl:R-EU_0411/3V -> rcl:R-EU_R1206
Connections:
- removed net D5: C4.1, C5.2, R31.2
- removed net N$20: Q3.G, R32.1
- removed net N$21: Q4.G, R33.1
- removed net N$22: Q5.G, R34.1
- removed net N$23: Q6.G, R35.1
- removed net N$24: C5.1, C6.2, R30.2
- removed net N$26: C3.1, C4.2, R32.2
- removed net N$27: C2.1, C3.2, R33.2
- removed net N$28: C1.1, C2.2, R34.2
- removed net N$29: C1.2, C7.2, R35.2
- new net CELL0: C6.2, Q6.S, R31.1
- new net CLK: U$1.CLK
- new net CLK_OUT: U$1.CLK_OUT
- new net CS_N: U$1.CS_N
- new net CS_N_OUT: U$1.CS_N_OUT
- new net DISCH1: R30.1, U$1.DISCH1
- new net DISCH2: R25.1, U$1.DISCH2
- new net DISCH3: R20.1, U$1.DISCH3
- new net DISCH4: R15.1, U$1.DISCH4
- new net DISCH5: R10.1, U$1.DISCH5
- new net DISCH6: R5.1, U$1.DISCH6
- new net IRQ: U$1.IRQ
- new net IRQ_IN: U$1.IRQ_IN
- new net MISO: U$1.MISO
- new net MISO_IN: U$1.MISO_IN
- new net MOSI: U$1.MOSI
- new net MOSI_OUT: U$1.MOSI_OUT
- new net N$10: Q5.G, R25.2
- new net N$12: Q6.G, R30.2
- new net N$3: Q2.D, R6.1, R7.1, R8.1, R9.1
- new net N$5: Q3.D, R11.1, R12.1, R13.1, R14.1
- new net N$7: Q4.D, R16.1, R17.1, R18.1, R19.1
- new net SCK: U$1.SCK
- new net SCK_OUT: U$1.SCK_OUT
- new net VDD: SJ1.3
- net CELL1: now also C5.2, C6.1, Q5.S, R26.2, R27.2, R28.2, R29.2, U$1.MBAT2; no longer JP6.1, R21.2, R22.2, R23.2, R24.2, R29.1
- net CELL2: now also C4.2, C5.1, Q4.S, R21.2, R22.2, R23.2, R24.2, U$1.MBAT3; no longer JP5.1, R17.2, R18.2, R19.2, R20.2, R28.1
- net CELL3: now also C3.2, C4.1, Q3.S, R17.2, R18.2, R19.2, U$1.MBAT4; no longer JP4.1, R13.2, R14.2, R15.2, R27.1
- net CELL4: now also C2.2, C3.1, Q2.S, R13.2, R14.2, U$1.MBAT5; no longer JP3.1, R10.2, R26.1, R9.2
- net CELL5: now also C1.2, C2.1, Q1.S, R9.2, U$1.MBAT6; no longer JP2.1, R25.1, R5.2
- net CELL6: now also C1.1, R32.2, U$1.MBAT7; no longer JP1.1, R36.1
- net GND: now also F1.2, R35.2, SJ1.1, U$1.AVSS, U$1.CS_FUSE, U$1.DVSS, U$1.GND, U$1.SCANMODE, U$1.TEMPVSS, U$1.VDDFUSE; no longer C7.1, JP7.1, Q6.S
- net N$11: now also R26.1, R27.1, R28.1, R29.1; no longer R21.1, R22.1, R23.1, R24.1
- net N$13: now also R31.2, U$1.MBAT1; no longer Q2.S, R26.2
- net N$14: now also R32.1, U$1.VDDHV; no longer Q3.S, R27.2
- net N$15: now also R33.2, R34.2, U$1.TEMPREF; no longer Q4.S, R28.2
- net N$16: now also R33.1, U$1.TEMP2; no longer Q5.S, R29.2
- net N$17: now also F1.1, R34.1, U$1.TEMP1; no longer Q1.G, R30.1
- net N$18: now also R35.1, U$1.BIASRES; no longer Q1.S, R25.2
- net N$19: now also SJ1.2, U$1.MFIRST; no longer Q2.G, R31.1
- net N$2: now also Q1.G, R5.2; no longer C6.1, R36.2
- net N$4: now also Q2.G, R10.2; no longer Q2.D, R5.1, R6.1, R7.1, R8.1
- net N$6: now also Q3.G, R15.2; no longer Q3.D, R10.1, R11.1, R12.1, R9.1
- net N$8: now also Q4.G, R20.2; no longer Q4.D, R13.1, R14.1, R15.1, R16.1
- net N$9: now also R21.1, R22.1, R23.1, R24.1; no longer R17.1, R18.1, R19.1, R20.1
Other:
- moved on the sheet: C1, C2, C3, C4, C5, C6, Q1, Q2, Q3, Q4, Q5, Q6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

Commit message: first working prototype
Parts:
- added R36: (no value), resistor:R-EU_R0805
- added U$2: TCMT1103-OPTO, SparkFun-DiscreteSemi:TCMT1103-OPTO
- added X1, X2: FH12-12S-0.5SH, con-hirose:FH12-12S-0.5SH
Connections:
- removed net N$14: R32.1, U$1.VDDHV
- new net OPTO_HI: U$2.A, X1-11.1, X2-11.1
- new net OPTO_LOW: U$2.K, X1-12.1, X2-12.1
- new net PD_N: U$1.PD_N, U$2.E
- new net VDDHV: R32.1, U$1.VDDHV, U$2.C
- new net VDDHVM: U$1.VDDHVM, X2-7.1
- new net VDDHVP: U$1.VDDHVP, X1-7.1
- net CELL0: now also R36.2
- net CLK: now also X2-2.1
- net CLK_OUT: now also X1-2.1
- net CS_N: now also X2-3.1
- net CS_N_OUT: now also X1-3.1
- net GND: now also R36.1
- net IRQ: now also X2-1.1
- net IRQ_IN: now also X1-1.1
- net MISO: now also X2-6.1
- net MISO_IN: now also X1-6.1
- net MOSI: now also X2-5.1
- net MOSI_OUT: now also X1-5.1
- net SCK: now also X2-4.1
- net SCK_OUT: now also X1-4.1
- net VDD: now also U$1.AVDD, U$1.DVDD, U$1.POW_ENA
